Commit message: Simple Controller add

File: robot_description/urdf/bumperbot_gazebo.urdf.xacro (robot description, xacro)
@@ -1,5 +1,5 @@
 <?xml version="1.0"?>
 <robot xmlns:xacro="https://www.ros.org/wiki/xacro">
-    <gazebo reference = "right_wheel_link">
+    <gazebo reference = "base_right_joint">
         <mu1>100000000000000.0</mu1>
         <mu2>100000000000000.0</mu2>
@@ -10,5 +10,5 @@
         <fdir1>1 0 0</fdir1>
     </gazebo>
-    <gazebo reference = "left_wheel_link">
+    <gazebo reference = "base_left_joint">
         <mu1>100000000000000.0</mu1>
         <mu2>100000000000000.0</mu2>
@@ -19,5 +19,5 @@
         <fdir1>1 0 0</fdir1>
     </gazebo>
-    <gazebo reference = "caster_front_link">
+    <gazebo reference = "base_front_caster_joint">
         <mu1>0.1</mu1>
         <mu2>0.1</mu2>
@@ -27,5 +27,5 @@
         <maxVel>0.1</maxVel>
     </gazebo>
-    <gazebo reference = "caster_rear_link">
+    <gazebo reference = "base_rear_caster_joint">
         <mu1>0.1</mu1>
         <mu2>0.1</mu2>
@@ -36,8 +36,8 @@
     </gazebo>
     <gazebo>
-        <!-- This plugin is for ROS2 Humble -->
+        <!-- This plugin is for ROS2 Humble or older -->
         <xacro:if value = "$(arg is_ignition)">
             <plugin filename = "ign_ros2_control-system" name = "ign_ros2_control::IgnitionROS2ControlPlugin">
-                <parameters></parameters>
+                <parameters>$(find robot_bringup)/config/bumperbot_controller.yaml</parameters>
             </plugin>
         </xacro:if>
@@ -45,5 +45,5 @@
         <xacro:unless value = "$(arg is_ignition)">
             <plugin filename = "gz_ros2_control-system" name = "gz_ros2_control::GazeboSimROS2ControlPlugin">
-                <parameters></parameters>
+                <parameters>$(find robot_bringup)/config/bumperbot_controller.yaml</parameters>
             </plugin>
         </xacro:unless>

File: robot_description/urdf/bumperbot_ros2_control.xacro (robot description, xacro)
@@ -3,5 +3,5 @@
     <ros2_control name = "RobotSystem" type = "system">
         <!-- This is for ROS2 Humble -->
-        <xacro:if value="$(args is_ignition)">
+        <xacro:if value="$(arg is_ignition)">
             <hardware>
                 <plugin>ign_ros2_control/IgnitionSystem</plugin>
@@ -9,10 +9,10 @@
         </xacro:if>
         <!-- This is for newer version of ROS2 -->
-        <xacro:unless value="$(args is_ignition)">
-            <hadrware>
+        <xacro:unless value="$(arg is_ignition)">
+            <hardware>
                 <plugin>gz_ros2_control/GazeboSimSystem</plugin>
-            </hadrware>
+            </hardware>
         </xacro:unless>
-        <joint name="right_wheel_link">
+        <joint name="base_right_joint">
             <!-- Data or command to the joint -->
             <command_interface name = "velocity">
@@ -24,5 +24,5 @@
             <state_interface name = "velocity"/>
         </joint>
-        <joint name="left_wheel_link">
+        <joint name="base_left_joint">
             <command_interface name = "velocity">
                 <param name = "min">-1</param>
