Commit message: Modify for Gazebo

File: robot_description/urdf/bumperbot_base.urdf.xacro (robot description, xacro)
@@ -1,4 +1,5 @@
 <?xml version="1.0"?>
-<robot name= "bumperbot" xmlns:xacro="https://www.ros.org/wiki/xacro">
+<robot xmlns:xacro="https://www.ros.org/wiki/xacro">
+    <xacro:arg name="is_ignition" default="false"/>
     <!-- ==================== Veriables ==================== -->
     <xacro:property name="base_length" value="0.9"/>
@@ -13,4 +14,11 @@
     <link name = "base_footprint"/>
     <link name = "base_link">
+        <inertial>
+        <origin xyz="0 0 0.04" rpy="0.0 0.25 0.3" />
+        <mass value="8.2573504e-01"/>
+        <inertia ixx="2.2124416e-02" ixy="-1.2294101e-04" ixz="3.4938785e-04"
+                 iyy="2.1193702e-02" iyz="-5.0120904e-05"
+                 izz="2.0064271e-02" />
+        </inertial>
         <visual>
             <geometry>
@@ -19,4 +27,10 @@
             <origin xyz = "0 0 0" rpy = "0 0 0"/>
         </visual>
+        <collision>
+            <geometry>
+                <mesh filename="package://robot_description/meshes/bumperbot/base_link.STL"/>
+            </geometry>
+            <origin xyz = "0 0 0" rpy = "0 0 0"/>
+        </collision>
     </link>
     <joint name = "base_joint" type = "fixed">
@@ -27,4 +41,11 @@
     <!-- ==================== right Wheel Link ==================== -->
     <link name = "right_wheel_link">
+        <inertial>
+        <origin xyz="0 -0.014 0" rpy="0 0 0" />
+        <mass value="0.0530086090966721" />
+        <inertia ixx="1.88176298336665E-05" ixy="-4.8444933029987E-10" ixz="1.88163708851143E-08"
+                 iyy="3.11510738647764E-05" iyz="-6.93560663069607E-11"
+                 izz="1.8801969558182E-05" />
+        </inertial>
         <visual>
             <geometry>
@@ -33,4 +54,10 @@
             <origin xyz = "0 0 0" rpy = "1.57 0 0"/>
         </visual>
+        <collision>
+            <geometry>
+                <sphere radius="0.033"/>
+            </geometry>
+            <origin xyz="0 -0.015 0" rpy="1.57 0 0"/>
+        </collision>
     </link>
     <joint name = "base_right_joint" type = "continuous">
@@ -42,4 +69,11 @@
     <!-- ==================== left Wheel Link ==================== -->
     <link name = "left_wheel_link">
+        <inertial>
+        <origin xyz="0 0.014 0" rpy="0 0 0" />
+        <mass value="0.0530086043217644" />
+        <inertia ixx="1.8792911368909E-05"  ixy="3.31256392204584E-10" ixz="-1.14082001662767E-08"
+                 iyy="3.11510738759073E-05" iyz="-3.60499245082192E-10"
+                 izz="1.88266886146847E-05" />
+        </inertial>
         <visual>
             <geometry>
@@ -48,4 +82,10 @@
             <origin xyz = "0 0 0" rpy = "-1.57 0 0"/>
         </visual>
+        <collision>
+            <geometry>
+                <sphere radius="0.033"/>
+            </geometry>
+            <origin xyz="0 0.015 0" rpy="1.57 0 0"/>
+        </collision>
     </link>
     <joint name = "base_left_joint" type = "continuous">
@@ -57,4 +97,11 @@
     <!-- ==================== Caster front Link ==================== -->
     <link name = "caster_front_link">
+        <inertial>
+        <origin xyz="3.89968128948481E-07 2.40073004698083E-07 0.00219173397061506" rpy="0 0 0" />
+        <mass value="1.44379265037903E-06" />
+        <inertia ixx="7.23075276010246E-11" ixy="-6.10956883467859E-16" ixz="2.22849693525031E-15"
+                 iyy="3.8713793085917E-11"  iyz="2.93909858781952E-15"
+                 izz="1.00967486676306E-10" />
+        </inertial>
         <visual>
             <geometry>
@@ -63,4 +110,10 @@
             <origin xyz = "0 0 0" rpy = "0 0 0"/>
         </visual>
+        <collision>
+            <geometry>
+                <sphere radius="0.005"/>
+            </geometry>
+            <origin xyz="0 0 0" rpy="0 0 0"/>
+        </collision>
     </link>
     <joint name = "base_front_caster_joint" type = "fixed">
@@ -71,4 +124,11 @@
     <!-- ==================== Caster rear Link ==================== -->
     <link name = "caster_rear_link">
+        <inertial>
+        <origin xyz="3.8996812895542E-07 2.40073004698083E-07 0.00219173397061509" rpy="0 0 0" />
+        <mass value="1.44379265037902E-06" />
+        <inertia ixx="7.23075276010246E-11" ixy="-6.10956872363424E-16" ixz="2.22849693527207E-15"
+                 iyy="3.87137930859167E-11" iyz="2.939098587861E-15"
+                 izz="1.00967486676306E-10" />
+        </inertial>
         <visual>
             <geometry>
@@ -77,4 +137,10 @@
             <origin xyz = "0 0 0" rpy = "0 0 0"/>
         </visual>
+        <collision>
+            <geometry>
+                <sphere radius="0.005"/>
+            </geometry>
+            <origin xyz="0 0 0" rpy="0 0 0"/>
+        </collision>
     </link>
     <joint name = "base_rear_caster_joint" type = "fixed">
@@ -83,3 +149,17 @@
         <origin xyz = "${-caster_wheel_seperation} 0 ${-caster_wheel_height}" rpy = "0 0 0" />
     </joint>
+    <!-- ==================== Cane Link ==================== -->
+    <!-- <link name = "can_link">
+        <visual>
+            <geometry>
+                <mesh filename="package://robot_description/meshes/bumperbot/can.STL"/>
+            </geometry>
+            <origin xyz = "-0.03 0.0325 0" rpy = "${pi/2.0} 0 0"/>
+        </visual>
+    </link>
+    <joint name = "base_can_joint" type = "fixed">
+        <parent link = "base_footprint" />
+        <child link = "can_link" />
+        <origin xyz = "0 0 0.111" rpy = "0 0 0" />
+    </joint> -->
 </robot>

Commit message: Joystick Controll add

File: robot_description/urdf/bumperbot_base.urdf.xacro (robot description, xacro)
@@ -3,7 +3,5 @@
     <xacro:arg name="is_ignition" default="false"/>
     <!-- ==================== Veriables ==================== -->
-    <xacro:property name="base_length" value="0.9"/>
-    <xacro:property name="base_width" value="0.4"/>
-    <xacro:property name="base_height" value="0.2"/>
+    <xacro:property name="wheel_radius" value="0.033"/>
     <xacro:property name="base_link_height" value="0.033"/>
     <xacro:property name="wheel_seperation" value="0.07"/>
@@ -56,5 +54,5 @@
         <collision>
             <geometry>
-                <sphere radius="0.033"/>
+                <sphere radius="${wheel_radius}"/>
             </geometry>
             <origin xyz="0 -0.015 0" rpy="1.57 0 0"/>
@@ -84,5 +82,5 @@
         <collision>
             <geometry>
-                <sphere radius="0.033"/>
+                <sphere radius="${wheel_radius}"/>
             </geometry>
             <origin xyz="0 0.015 0" rpy="1.57 0 0"/>

Commit message: collision issue solve

File: robot_description/urdf/bumperbot_base.urdf.xacro (robot description, xacro)
@@ -12,5 +12,5 @@
     <link name = "base_footprint"/>
     <link name = "base_link">
-        <inertial>
+        <!-- <inertial>
         <origin xyz="0 0 0.04" rpy="0.0 0.25 0.3" />
         <mass value="8.2573504e-01"/>
@@ -18,5 +18,6 @@
                  iyy="2.1193702e-02" iyz="-5.0120904e-05"
                  izz="2.0064271e-02" />
-        </inertial>
+        </inertial> -->
+        <xacro:cylinder_inertia m="2.0" r="0.075" l="0.105" o_xyz="0 0 0.028" o_rpy="0 0 0" />
         <visual>
             <geometry>
@@ -27,7 +28,8 @@
         <collision>
             <geometry>
-                <mesh filename="package://robot_description/meshes/bumperbot/base_link.STL"/>
+                <!-- <mesh filename="package://robot_description/meshes/bumperbot/base_link.STL"/> -->
+                <cylinder radius="0.075" length="0.105"/>
             </geometry>
-            <origin xyz = "0 0 0" rpy = "0 0 0"/>
+            <origin xyz = "0 0 0.028" rpy = "0 0 0"/>
         </collision>
     </link>

File: robot_description/urdf/bumperbot_complete.urdf.xacro (robot description, xacro)
@@ -2,4 +2,5 @@
 <robot name= "bumperbot" xmlns:xacro="https://www.ros.org/wiki/xacro">
     <xacro:include filename="$(find robot_description)/urdf/common_materials.xacro"/>
+    <xacro:include filename="$(find robot_description)/urdf/common_properties.urdf.xacro"/>
     <xacro:include filename="$(find robot_description)/urdf/bumperbot_ros2_control.xacro"/>
     <xacro:include filename="$(find robot_description)/urdf/bumperbot_gazebo.urdf.xacro"/>
